File: Hardware/instrumentation_amplifier.kicad_sch (KiCad schematic)
At the start: 13 parts, among them U1 INA128

Commit message: completed hardware
Changed lines of the file:
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@@
 	(wire
 		(pts
-			(xy 25.4 63.5) (xy 30.48 63.5)
+			(xy 19.05 63.5) (xy 30.48 63.5)
 		)
 		(stroke
@@
 	(wire
 		(pts
-			(xy 25.4 52.07) (xy 30.48 52.07)
+			(xy 19.05 52.07) (xy 30.48 52.07)
 		)
 		(stroke
@@
 	(wire
 		(pts
-			(xy 25.4 52.07) (xy 25.4 63.5)
+			(xy 19.05 52.07) (xy 19.05 63.5)
 		)
 		(stroke
@@
 			(width 0)
 			(type default)
+		)
+	)
+	(label "INA128_Output"
+		(at 124.46 62.23 0)
+		(effects
+			(font
+				(size 1.27 1.27)
+			)
+			(justify left bottom)
+		)
+	)
+	(label "INA128_input"
+		(at 19.05 52.07 0)
+		(effects
+			(font
+				(size 1.27 1.27)
+			)
+			(justify left bottom)
 		)
 	)
@@
 	(hierarchical_label "In"
 		(shape output)
-		(at 25.4 55.88 180)
+		(at 19.05 55.88 180)
 		(effects
 			(font
@@
 			(at 114.3 62.23 0)
 			(hide yes)
+			(show_name no)
+			(do_not_autoplace no)
+			(effects
+				(font
+					(size 1.27 1.27)
+				)
+			)
+		)
+		(property "Sim.Library" "spice\\sbom763\\INA128_TINA_AIO\\INA128.LIB"
+			(at 114.3 62.23 0)
+			(hide yes)
+			(show_name no)
+			(do_not_autoplace no)
+			(effects
+				(font
+					(size 1.27 1.27)
+				)
+			)
+		)
+		(property "Sim.Name" "INA128"
+			(at 114.3 62.23 0)
+			(hide yes)
+			(show_name no)
+			(do_not_autoplace no)
+			(effects
+				(font
+					(size 1.27 1.27)
+				)
+			)
+		)
+		(property "Sim.Device" "SUBCKT"
+			(at 114.3 62.23 0)
+			(hide yes)
+			(show_name no)
+			(do_not_autoplace no)
+			(effects
+				(font
+					(size 1.27 1.27)
+				)
+			)
+		)
+		(property "Sim.Pins" "1=1 2=2 3=3 4=4 5=5 6=8 7=9 8=10"
+			(at 114.3 62.23 0)
+			(hide yes)
