File: Hardware/signal_conditioning.kicad_sch (KiCad schematic)
At the start: 4 parts, among them T1 SCT-013-000

Commit message: completed hardware
Parts:
- added V2: VSIN, symbol Simulation_SPICE:VSIN
Connections:
- net GND: now also V2.2; no longer V1.2
- new net: V1.2, V2.1
